Commit message: feat: add manual robot placement workflow

File: dentobot_description/urdf/dentobot.urdf (robot description, URDF)
Before this commit: robot dentobot, 8 links, 7 joints
Joints:
- joint base_link_to_link-1: origin xyz=0.0 0.0 0.0 rpy=0.0 0.0 0.0 -> xyz=0.0 0.0 0.0 rpy=-1.5707963267948966 0.0 0.0
- joint link-1_Revolute-1: limit lower=0.0 upper=6.283185 effort=1000000 velocity=1000000 -> lower=-0.44296456415616081 upper=5.8402204358438388 effort=1000000 velocity=1000000; origin xyz=0.0 0.0 0.0 rpy=1.5707963267948966 -0.0 0.0 -> xyz=0.0 0.0 0.0 rpy=1.570796326794897 -0.4429645641561608 2.90490637318374e-17
- joint link-3_Revolute-3: limit lower=0.0 upper=6.283185 effort=1000000 velocity=1000000 -> lower=-1.0901326507956584 upper=5.1930523492043417 effort=1000000 velocity=1000000; origin xyz=-0.047122859999999996 -0.11 -0.09383196 rpy=-3.141592653589793 1.5707963267948966 0 -> xyz=-0.047122859999999996 -0.11 -0.09383196 rpy=2.067357736975897 1.101119703255167 -2.067357736975897
- joint link-4_Slider-4: axis 0.893638 2.4694080114073816e-17 -0.44878900000000005 -> -0.893638 -2.4694080114073816e-17 0.44878900000000005
- joint link-5_Revolute-5: limit lower=0.0 upper=6.283185 effort=1000000 velocity=1000000 -> lower=-0.018849555921538759 upper=6.2643354440784611 effort=1000000 velocity=1000000; origin xyz=-0.021752659999999997 -0.006762529999999991 0.007295090000000003 rpy=5.551115123125784e-17 -1.5707963267948966 0 -> xyz=-0.021752659999999997 -0.006762529999999991 0.007295090000000003 rpy=-2.933237124130466 -1.553411074346388 2.925952888262058
- joint pneumatic_spindle-Copy_Revolute-6: origin xyz=0.035401760000000004 0.0029788100000000027 0.04568638 rpy=-3.141592653589793 1.5707963267948966 0 -> xyz=0.035401760000000004 0.0029788100000000027 0.04568638 rpy=0.9502765943544816 1.0092142015761 -1.935369066862216

Commit message: feat: checkpoint workflow simulation and case persistence

File: dentobot_description/urdf/dentobot.urdf (robot description, URDF)
Before this commit: robot dentobot, 8 links, 7 joints
Links:
- added link dentobot_tool_tcp
Joints:
- added joint burr_to_dentobot_tool_tcp: type fixed, parent burr, child dentobot_tool_tcp, origin xyz=0.0 0.0 0.0 rpy=-2.61089174 -0.36458195 -0.20627347

Commit message: feat: implement native gated Step 6 simulation workflow

File: dentobot_description/urdf/dentobot.urdf (robot description, URDF)
Before this commit: robot dentobot, 9 links, 8 joints
Links:
- added link dentobot_drill_tip_provisional
Joints:
- added joint dentobot_tool_tcp_to_drill_tip_provisional: type fixed, parent dentobot_tool_tcp, child dentobot_drill_tip_provisional, origin xyz=0.0 0.0 0.007 rpy=0.0 0.0 0.0

Commit message: Document and sync Goal 1 stabilization

File: dentobot_description/urdf/dentobot.urdf (robot description, URDF)
Before this commit: robot dentobot, 10 links, 9 joints
Joints:
- joint link-2_Slider-2: axis 0.0 0.9999999999999999 0.0 -> 0.0 -0.9999999999999999 0.0; origin xyz=0.0 0.0 0.08 rpy=-1.5707963267948966 -0.0 1.5707963267948966 -> xyz=0.0 0.0 0.0 rpy=-1.5707963267948966 -0.0 1.5707963267948966
- joint link-5_Revolute-5: limit lower=-0.018849555921538759 upper=6.2643354440784611 effort=1000000 velocity=1000000 -> effort=1000000 velocity=1000000; type revolute -> continuous

Commit message: feat(step6): remove spindle from MoveIt planning model

File: dentobot_description/urdf/dentobot.urdf (robot description, URDF)
Before this commit: robot dentobot, 10 links, 9 joints
Links:
- added link dentobot_drill_tcp
Joints:
- added joint pneumatic_spindle-Copy_to_dentobot_drill_tcp: type fixed, parent pneumatic_spindle-Copy, child dentobot_drill_tcp, origin xyz=0.041042122156006 -0.000048165096147 0.042853759920214 rpy=-2.224555444403231 0.842809592516694 -2.582877942399306

Commit message: feat(step6): checkpoint guarded planning and case workflows
Checkpoint the current simulation-only Step 6 work: phased collision guarding and diagnostics, bounded tool/guide contact warnings, 1 mm burr model, capped insertion evidence, retraction/Home support, segmentation-run isolation, case lifecycle hardening, assisted pulp endpoint and guide-shell geometry, launch/setup updates, verification routing, and controlled records.\n\nVerification: 106 focused tests passed; 40 changed Python files compiled; UI XML, verification JSON, shell syntax, and git diff checks passed. Full exact-case approach/drilling/retraction/Home acceptance remains open because adjacent FDI21 geometry and monitored-state convergence still require resolution.

File: dentobot_description/urdf/dentobot.urdf (robot description, URDF)
Before this commit: robot dentobot, 11 links, 10 joints
Links:
- link burr: geometry collision mesh filename=package://dentobot_description/meshes/burr_simulation_1mm.s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 scale=0.001 0.001 0.001; visual mesh filename=package://dentobot_description/meshes/burr_simulation_1mm.s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 scale=0.001 0.001 0.001
