Commit message: Checkpoint Step 6 five-DOF workbench and meeting evidence

File: dentobot_description/urdf/dentobot.diagnostic-no-spindle-collision.urdf (robot description, URDF)
Before this commit: robot dentobot, 11 links, 10 joints
Joints:
- removed joint pneumatic_spindle-Copy_Revolute-6
- added joint pneumatic_spindle-Copy_to_burr_fixed: type fixed, parent pneumatic_spindle-Copy, child burr, origin xyz=0.035401760000000004 0.0029788100000000027 0.04568638 rpy=0.9502765943544816 1.0092142015761 -1.935369066862216

File: dentobot_description/urdf/dentobot.urdf (robot description, URDF)
Before this commit: robot dentobot, 11 links, 10 joints
Joints:
- removed joint pneumatic_spindle-Copy_Revolute-6
- added joint pneumatic_spindle-Copy_to_burr_fixed: type fixed, parent pneumatic_spindle-Copy, child burr, origin xyz=0.035401760000000004 0.0029788100000000027 0.04568638 rpy=0.9502765943544816 1.0092142015761 -1.935369066862216
